Commit message: a7 attempt

File: body.urdf (robot description, URDF)
Before this commit: robot robot, 9 links, 8 joints
Links:
- removed link BackLeg
- removed link BackLowerLeg
- removed link FrontLeg
- removed link FrontLowerLeg
- removed link LeftLeg
- removed link LeftLowerLeg
- removed link RightLeg
- removed link RightLowerLeg
- removed link Torso
- added link Head, mass 1; collision box size=1 1 1; visual box size=1 1 1
- added link Seg-0, mass 1; collision box size=0.16217429503691094 0.37597697941900154 0.27616505500849875; visual box size=0.16217429503691094 0.37597697941900154 0.27616505500849875
- added link Seg-1, mass 1; collision box size=0.42162040857670813 0.677080188845371 0.860451909822161; visual box size=0.42162040857670813 0.677080188845371 0.860451909822161
- added link Seg-2, mass 1; collision box size=0.9256801469605592 0.5893086604978275 0.057921964797602477; visual box size=0.9256801469605592 0.5893086604978275 0.057921964797602477
- added link Seg-3, mass 1; collision box size=0.9518589426364817 0.4168280013850829 0.35671168118265806; visual box size=0.9518589426364817 0.4168280013850829 0.35671168118265806
- added link Seg-4, mass 1; collision box size=0.4755156181415202 0.7883785505719364 0.6497587420972728; visual box size=0.4755156181415202 0.7883785505719364 0.6497587420972728
- added link Seg-5, mass 1; collision box size=0.2154375759059085 0.2987140348052182 0.9879370287892457; visual box size=0.2154375759059085 0.2987140348052182 0.9879370287892457
- added link Seg-6, mass 1; collision box size=0.48384060487597336 0.3230728477064211 0.2413699698051529; visual box size=0.48384060487597336 0.3230728477064211 0.2413699698051529
Joints:
- removed joint BackLeg_BackLowerLeg
- removed joint FrontLeg_FrontLowerLeg
- removed joint LeftLeg_LeftLowerLeg
- removed joint RightLeg_RightLowerLeg
- removed joint Torso_BackLeg
- removed joint Torso_FrontLeg
- removed joint Torso_LeftLeg
- removed joint Torso_RightLeg
- added joint Head_Seg-0: type revolute, parent Head, child Seg-0, origin xyz=0.5 0.5 0 rpy=0 0 0, axis 1 0 0, limit lower=-3.14159 upper=3.14159 effort=0.0 velocity=0.0
- added joint Seg-0_Seg-1: type revolute, parent Seg-0, child Seg-1, origin xyz=0.08108714751845547 0.0 0.0 rpy=0 0 0, axis 0 0 1, limit lower=-3.14159 upper=3.14159 effort=0.0 velocity=0.0
- added joint Seg-1_Seg-2: type revolute, parent Seg-1, child Seg-2, origin xyz=0.21081020428835406 0.3385400944226855 0.860451909822161 rpy=0 0 0, axis 0 1 0, limit lower=-3.14159 upper=3.14159 effort=0.0 velocity=0.0
- added joint Seg-2_Seg-3: type revolute, parent Seg-2, child Seg-3, origin xyz=0.4628400734802796 0.29465433024891374 0.057921964797602477 rpy=0 0 0, axis 1 0 0, limit lower=-3.14159 upper=3.14159 effort=0.0 velocity=0.0
- added joint Seg-3_Seg-4: type revolute, parent Seg-3, child Seg-4, origin xyz=0.47592947131824087 0.20841400069254146 0.35671168118265806 rpy=0 0 0, axis 0 0 1, limit lower=-3.14159 upper=3.14159 effort=0.0 velocity=0.0
- added joint Seg-4_Seg-5: type revolute, parent Seg-4, child Seg-5, origin xyz=0.0 0.3941892752859682 0.6497587420972728 rpy=0 0 0, axis 0 1 0, limit lower=-3.14159 upper=3.14159 effort=0.0 velocity=0.0
- added joint Seg-5_Seg-6: type revolute, parent Seg-5, child Seg-6, origin xyz=0.10771878795295425 0.0 0.0 rpy=0 0 0, axis 0 0 1, limit lower=-3.14159 upper=3.14159 effort=0.0 velocity=0.0
